File: EAGLE/HTSenti/htsenti.brd (EAGLE design)
At the start: 100 x 80 mm, 15 parts, among them J1 NANO_FOOTPRINT

Commit message: MVP PCB
Parts:
- moved R1 141.2 mm to (88.9, 4.45)
- moved LED1 126.7 mm to (95.2, 3.81)
- moved R3 120.4 mm to (88.9, 2.54)
- moved R4 118.9 mm to (69.8, 5.08), turned to 90 degrees
- moved R2 115.3 mm to (88.9, 6.35)
- moved DHT22 106.6 mm to (66.0, 7.62), turned to 90 degrees
- moved J1 80.7 mm to (50.8, 55.9)
- moved U$1 53.3 mm to (10.2, 7.62)
- moved U$3 6.35 mm to (95.2, 76.2)
- moved U$5 6.35 mm to (3.81, 76.2)
- moved JP3 6.35 mm to (95.2, 45.7)
- moved JP4 6.35 mm to (4.32, 45.7)
- moved U$6 6.35 mm to (29.2, 38.4)
- moved U$2 6.35 mm to (95.2, 15.2)
- moved U$4 6.35 mm to (3.81, 15.2)
Routing:
- net GND: track 0.00 -> 6.90 mm, vias 0 -> 1
- net N$7: track 0.00 -> 3.94 mm
- net +5V: track 0.00 -> 3.94 mm
- net N$2: track 0.00 -> 3.85 mm
- net N$1: track 0.00 -> 3.76 mm
- net N$3: track 0.00 -> 3.68 mm
Other:
- outline, holes or cut-outs redrawn
- board text removed: "CD"
